Commit message: Update physical robot parameters (wheel radius 70mm, track width 370mm), restore silky smooth S-curve, and verify SLAM mapping

File: src/amr_assembly_description/urdf/amr_assembly_description.urdf (robot description, URDF)
Before this commit: robot amr_assembly, 13 links, 12 joints
Links:
- link left_wheel: geometry collision cylinder length=0.050 radius=0.070; visual mesh filename=package://amr_assembly_description/meshes/wheel_1_2.dae
- link right_wheel: geometry collision cylinder length=0.050 radius=0.070; visual mesh filename=package://amr_assembly_description/meshes/wheel_1.dae
Joints:
- joint left_wheel_joint: origin xyz=0 0.2135 0.025 rpy=0 0 3.14159265359 -> xyz=0 0.185 0.015 rpy=0 0 3.14159265359
- joint right_wheel_joint: origin xyz=0 -0.2135 0.025 rpy=0 0 3.14159265359 -> xyz=0 -0.185 0.015 rpy=0 0 3.14159265359

Commit message: Refactor robot URDF, wheel joints, TF frames, and Nav2 footprint to canonical ROS orientation

File: src/amr_assembly_description/urdf/amr_assembly_description.urdf (robot description, URDF)
Before this commit: robot amr_assembly, 13 links, 12 joints
Joints:
- joint left_wheel_joint: axis 0 -1 0 -> 0 1 0; origin xyz=0 0.185 0.015 rpy=0 0 3.14159265359 -> xyz=0 0.185 0.015 rpy=0 0 0
- joint right_wheel_joint: axis 0 -1 0 -> 0 1 0; origin xyz=0 -0.185 0.015 rpy=0 0 3.14159265359 -> xyz=0 -0.185 0.015 rpy=0 0 0

Commit message: Update chassis orientation (90 deg) and drive wheels to Y=±0.235m (W=0.470m) matching real AMR hardware

File: src/amr_assembly_description/urdf/amr_assembly_description.urdf (robot description, URDF)
Before this commit: robot amr_assembly, 13 links, 12 joints
Joints:
- joint caster_wheel1_joint: origin xyz=0.120775 0.117491 -0.007140912 rpy=1.5707963 0 -1.5707963 -> xyz=0.1174 0.1208 -0.007140912 rpy=1.5707963 0 0
- joint caster_wheel2_joint: origin xyz=-0.149932 -0.117423 -0.007140912 rpy=1.5707963 0 -1.5707963 -> xyz=-0.1174 -0.1499 -0.007140912 rpy=1.5707963 0 0
- joint caster_wheel3_joint: origin xyz=0.121583 -0.117333 -0.007140912 rpy=1.5707963 0 -1.5707963 -> xyz=0.1174 -0.1499 -0.007140912 rpy=1.5707963 0 0
- joint caster_wheel4_joint: origin xyz=-0.149381 0.116260 -0.007140912 rpy=1.5707963 0 -1.5707963 -> xyz=-0.1174 0.1208 -0.007140912 rpy=1.5707963 0 0
- joint left_wheel_joint: origin xyz=0 0.185 0.015 rpy=0 0 0 -> xyz=0 0.235 0.015 rpy=0 0 0
- joint right_wheel_joint: origin xyz=0 -0.185 0.015 rpy=0 0 0 -> xyz=0 -0.235 0.015 rpy=0 0 0

Commit message: Align LiDAR (X=0.180m, Z=0.760m) and Camera (X=0.215m, Z=0.157m) cleanly onto the front chassis beams

File: src/amr_assembly_description/urdf/amr_assembly_description.urdf (robot description, URDF)
Before this commit: robot amr_assembly, 13 links, 12 joints
Joints:
- joint camera_joint: origin xyz=0.241580 0.009331 0.156845974 rpy=1.79844 0 1.5707963 -> xyz=0.215 0.0 0.156845974 rpy=1.79844 0 1.5707963
- joint lidar_joint: origin xyz=0.192495 -0.003059 0.760213094 rpy=1.5707963 0 3.14159265359 -> xyz=0.180 0.0 0.760213094 rpy=1.5707963 0 3.14159265359
